Commit message: Task 1

File: rb1_ros2_description/xacro/rb1_ros2_base.urdf.xacro (robot description, xacro)
@@ -114,13 +114,4 @@
             <state_interface name="effort"/>
         </joint>
-        <joint name="robot_elevator_platform_joint">
-            <command_interface name="effort">
-            <param name="min">0</param>
-            <param name="max">10</param>
-            </command_interface>
-            <state_interface name="position"/>
-            <state_interface name="velocity"/>
-            <state_interface name="effort"/>
-        </joint>
     </ros2_control>
     <gazebo>

Commit message: Task2

File: rb1_ros2_description/xacro/rb1_ros2_base.urdf.xacro (robot description, xacro)
@@ -114,4 +114,13 @@
             <state_interface name="effort"/>
         </joint>
+        <joint name="robot_elevator_platform_joint">
+            <command_interface name="effort">
+            <param name="min">0</param>
+            <param name="max">10</param>
+            </command_interface>
+            <state_interface name="position"/>
+            <state_interface name="velocity"/>
+            <state_interface name="effort"/>
+        </joint>
     </ros2_control>
     <gazebo>
